File: EduboardV2_ATmega328PB.kicad_pcb (KiCad board)
At the start: 4 copper layers, 35 x 63.3 mm, 21 parts, among them J1 EduboardV2 PCIE UP Board Conn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, Q3 AO3401A, SW1 K2-1102SP-C4SC-04, U5 LD1117S33TR_SOT223

Commit message: schematic done. layout done aswell. Have to check everything trice
Parts:
- removed C17: 100n, Capacitor_SMD:C_0603_1608Metric
- added C1: 100n, Capacitor_SMD:C_0402_1005Metric, F.Cu at (112.2, 113.6)
- added C10: 100n, Capacitor_SMD:C_0402_1005Metric, F.Cu at (111.0, 134.1)
- added C11: 100n, Capacitor_SMD:C_0402_1005Metric, F.Cu at (124.9, 134.9)
- added C2: 100n, Capacitor_SMD:C_0402_1005Metric, F.Cu at (121.4, 107.8)
- added C3: 100n, Capacitor_SMD:C_0402_1005Metric, F.Cu at (124.0, 116.0)
- added C4: 100n, Capacitor_SMD:C_0402_1005Metric, F.Cu at (115.6, 107.8)
- added C5: 100n, Capacitor_SMD:C_0402_1005Metric, F.Cu at (117.6, 119.6)
- added C6: 12p, Capacitor_SMD:C_0402_1005Metric, F.Cu at (121.2, 123.2)
- added C7: 12p, Capacitor_SMD:C_0402_1005Metric, F.Cu at (127.2, 123.2)
- added C8: 100n, Capacitor_SMD:C_0402_1005Metric, F.Cu at (115.7, 119.6)
- added C9: 100n, Capacitor_SMD:C_0402_1005Metric, F.Cu at (111.0, 132.5)
- added J2: JTAG_mEDBG, Connector_PinHeader_2.54mm:PinHeader_2x05_P2.54mm_Vertical, F.Cu at (118.8, 98.5)
- added JP1: SolderJumper_2_Open, Jumper:SolderJumper-2_P1.3mm_Bridged_RoundedPad1.0x1.5mm, F.Cu at (126.5, 109.0)
- added JP16: SolderJumper_3_Bridged12, EduboardV2_kicadlib:SolderJumper_Small-3_bridged12, B.Cu at (113.8, 133.2)
- added JP17: SolderJumper_3_Bridged12, EduboardV2_kicadlib:SolderJumper_Small-3_bridged12, B.Cu at (116.8, 133.2)
- added JP18: SolderJumper_3_Bridged12, EduboardV2_kicadlib:SolderJumper_Small-3_bridged12, B.Cu at (119.9, 133.2)
- added JP19: SolderJumper_3_Bridged12, EduboardV2_kicadlib:SolderJumper_Small-3_bridged12, B.Cu at (123.0, 133.2)
- added JP2: SolderJumper_3_Bridged12, EduboardV2_kicadlib:SolderJumper_Small-3_bridged12, B.Cu at (122.0, 141.7)
- added JP20: SolderJumper_3_Bridged12, EduboardV2_kicadlib:SolderJumper_Small-3_bridged12, B.Cu at (126.0, 133.2)
- added JP21: SolderJumper_3_Bridged12, EduboardV2_kicadlib:SolderJumper_Small-3_bridged12, B.Cu at (129.1, 133.2)
- added JP22: SolderJumper_3_Bridged12, EduboardV2_kicadlib:SolderJumper_Small-3_bridged12, B.Cu at (129.8, 124.7)
- added JP23: SolderJumper_3_Bridged12, EduboardV2_kicadlib:SolderJumper_Small-4_bridged14, B.Cu at (106.8, 141.8)
- added JP3: SolderJumper_3_Bridged12, EduboardV2_kicadlib:SolderJumper_Small-3_bridged12, B.Cu at (119.0, 141.7)
- added JP30: SolderJumper_3_Bridged12, EduboardV2_kicadlib:SolderJumper_Small-3_bridged12, B.Cu at (117.7, 124.7)
- added JP34: SolderJumper_3_Bridged12, EduboardV2_kicadlib:SolderJumper_Small-3_bridged12, B.Cu at (114.7, 124.7)
- added JP4: SolderJumper_3_Bridged12, EduboardV2_kicadlib:SolderJumper_Small-4_bridged14, B.Cu at (109.8, 141.8)
- added JP5: SolderJumper_3_Bridged12, EduboardV2_kicadlib:SolderJumper_Small-3_bridged12, B.Cu at (112.9, 141.7)
- added JP6: SolderJumper_3_Bridged12, EduboardV2_kicadlib:SolderJumper_Small-3_bridged12, B.Cu at (115.9, 141.7)
- added JP7: SolderJumper_3_Bridged12, EduboardV2_kicadlib:SolderJumper_Small-3_bridged12, B.Cu at (125.0, 141.7)
- added JP8: SolderJumper_2_Open, Jumper:SolderJumper-2_P1.3mm_Bridged_RoundedPad1.0x1.5mm, F.Cu at (126.5, 114.0)
- added LED1: 19-217/BHC-ZL1M2RY/3T, EduboardV2_kicadlib:LED0603-FD_BLUE, F.Cu at (130.7, 111.7)
- added R1: 100k, Resistor_SMD:R_0402_1005Metric, F.Cu at (128.9, 109.7)
- added R10: 1k, Resistor_SMD:R_0402_1005Metric, F.Cu at (118.3, 143.2)
- added R11: 330R, Resistor_SMD:R_0603_1608Metric, F.Cu at (123.9, 112.2)
- added R12: 3k3, Resistor_SMD:R_0402_1005Metric, F.Cu at (127.9, 111.7)
- added R13: 100k, Resistor_SMD:R_0402_1005Metric, F.Cu at (116.6, 119.6)
- added R2: 3k3, Resistor_SMD:R_0402_1005Metric, F.Cu at (127.8, 116.5)
- added R3: 0R, Resistor_SMD:R_0603_1608Metric, F.Cu at (126.0, 117.3)
- added R4: 330R, Resistor_SMD:R_0603_1608Metric, F.Cu at (111.2, 120.2)
- added R5: 330R, Resistor_SMD:R_0603_1608Metric, F.Cu at (112.8, 120.2)
- added R8: 330R, Resistor_SMD:R_0603_1608Metric, F.Cu at (114.3, 120.2)
- added R9: 1k, Resistor_SMD:R_0402_1005Metric, F.Cu at (121.3, 143.2)
- added U1: ATMEGA32U4-MU, EduboardV2_kicadlib:VQFN-44_L7.0-W7.0-P0.50-BL-EP5.2, F.Cu at (118.5, 113.5)
- added U2: ATMEGA328PB-AUR, EduboardV2_kicadlib:TQFP-32_L7.0-W7.0-P0.80-LS9.0-BL, F.Cu at (117.9, 134.5)
- added X1: M16000E067, EduboardV2_kicadlib:CRYSTAL-SMD_4P-L3.2-W2.5-BL, F.Cu at (124.2, 123.2)
- C26, C28: footprint Capacitor_SMD:C_0603_1608Metric -> Capacitor_SMD:C_0402_1005Metric
- R19, R6, R7: footprint Resistor_SMD:R_0603_1608Metric -> Resistor_SMD:R_0402_1005Metric
- R25: value 2k2 -> 3k3; footprint Resistor_SMD:R_0603_1608Metric -> Resistor_SMD:R_0402_1005Metric
- moved C27 61.6 mm to (106.5, 132.9), turned to 180 degrees
- moved C25 59.7 mm to (103.1, 118.5), turned to 180 degrees
- moved Q3 55.0 mm to (106.6, 135.8)
- moved D1 54.6 mm to (102.6, 102.8), turned to 180 degrees
- moved D3 53.5 mm to (103.7, 108.8)
- moved R19 51.3 mm to (129.1, 127.3), turned to -90 degrees
- moved D2 50.3 mm to (106.7, 108.8), turned to 180 degrees
- moved C28 48.8 mm to (105.8, 131.2), turned to 180 degrees
- moved U5 47.7 mm to (105.3, 126.0), turned to -90 degrees
- moved R25 47.1 mm to (107.8, 138.5), turned to -90 degrees
- moved C26 46.6 mm to (102.7, 120.2), turned to 180 degrees
- moved SW1 45.6 mm to (131.3, 134.3)
- moved USBC1 39.7 mm to (111.5, 99.5), turned to 180 degrees
- moved R29 39.3 mm to (104.4, 115.0), turned to 90 degrees
- moved R31 39.3 mm to (104.4, 111.1), turned to -90 degrees
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Connections:
- net /DebugChip/D_N renamed USB_N
- net /DebugChip/D_P renamed USB_P
- net UP_Reset renamed ~{RESET_DW}
- J1 pad 11: unconnected-(J1-UART0_UP_RX-Pad11) -> Net-(J1-UART0_UP_RX)
- J1 pad 13: unconnected-(J1-UART1_RS485_TX-Pad13) -> UART1_TX
- J1 pad 15: unconnected-(J1-UART1_RS485_RX-Pad15) -> UART1_RX
- J1 pad 16: unconnected-(J1-RS485_DE-Pad16) -> RS485_DE
- J1 pad 17: unconnected-(J1-~{FLASH_CS}-Pad17) -> GPIO_FLASH_CS
- J1 pad 18: unconnected-(J1-~{General_Reset}-Pad18) -> ~{General_Reset}
- J1 pad 19: unconnected-(J1-~{SD_CS}-Pad19) -> GPIO_SD_CS
- J1 pad 20: unconnected-(J1-~{TFT_CS}-Pad20) -> LCD_CS
- J1 pad 22: unconnected-(J1-TFT_DC-Pad22) -> LCD_DC
- J1 pad 24: unconnected-(J1-SPI_SCK-Pad24) -> SPI_SCK
- J1 pad 26: unconnected-(J1-SPI_MISO-Pad26) -> SPI_MISO
- J1 pad 28: unconnected-(J1-SPI_MOSI-Pad28) -> SPI_MOSI
- J1 pad 29: unconnected-(J1-WS2812_Data-Pad29) -> GPIO_WS2812_DATA
- J1 pad 30: unconnected-(J1-SCL-Pad30) -> SCL
- J1 pad 32: unconnected-(J1-SDA-Pad32) -> SDA
- J1 pad 34: unconnected-(J1-GPIOX4/AN5/I2S_MCLK-Pad34) -> GPIOX4
- J1 pad 36: unconnected-(J1-GPIOX3/AN4/I2S_SCLK-Pad36) -> GPIOX3
- J1 pad 38: unconnected-(J1-GPIOX2/AN3/I2S_LRCK-Pad38) -> GPIOX2
- J1 pad 40: unconnected-(J1-GPIOX1/AN2/I2S_DIN-Pad40) -> GPIOX1
- J1 pad 42: unconnected-(J1-GPIOX0/AN1/I2S_DOUT-Pad42) -> GPIOX0
- J1 pad 44: unconnected-(J1-AN0/Pot0-Pad44) -> GPIO_AN0
- J1 pad 46: unconnected-(J1-SW0-Pad46) -> GPIO_SW0
- J1 pad 48: unconnected-(J1-SW1-Pad48) -> GPIO_SW1
- J1 pad 50: unconnected-(J1-SW2-Pad50) -> GPIO_SW2
- J1 pad 52: unconnected-(J1-SW3-Pad52) -> GPIO_SW3
- J1 pad 9: unconnected-(J1-UART0_UP_TX-Pad9) -> Net-(J1-UART0_UP_TX)
Routing:
- net +3V3: track 0.00 -> 150.7 mm, vias 0 -> 12
- net VBUS: track 0.00 -> 96.8 mm, vias 0 -> 4
- net GND: track 0.00 -> 85.9 mm, vias 0 -> 107
- net RS485_DE: track 0.00 -> 53.8 mm
- net UART1_TX: track 0.00 -> 46.2 mm, vias 0 -> 1
- net USB_Debug_D+: track 0.00 -> 45.2 mm, vias 0 -> 1
- net USB_Debug_D-: track 0.00 -> 45.2 mm, vias 0 -> 1
- net UART1_RX: track 0.00 -> 44.7 mm, vias 0 -> 1
- net SPI_MISO: track 0.00 -> 43.6 mm, vias 0 -> 3
- net SPI_SCK: track 0.00 -> 40.5 mm, vias 0 -> 2
- net ~{RESET_DW}: track 0.00 -> 40.2 mm
- net SPI_MOSI: track 0.00 -> 39.4 mm, vias 0 -> 3
- net GPIOX0: track 0.00 -> 38.8 mm
- net GPIO_SW0: track 0.00 -> 37.8 mm, vias 0 -> 1
- net GPIO_WS2812_DATA: track 0.00 -> 36.8 mm, vias 0 -> 2
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Other:
- board text added: "Eduboard2 UP-Board ATmega328PB V${HW_VERSION}"
- board text removed: "Eduboard2 UP-Board xxx V${HW_VERSION}"

Commit message: ready for order first prototype
Parts:
- added G***: LOGO, EduboardV2_kicadlib:logo_moonlander, F.Cu at (130.2, 124.0)
- added G***: LOGO, EduboardV2_kicadlib:logo3, F.Cu at (131.9, 102.9)
- added G***: LOGO, EduboardV2_kicadlib:JuventusLogo, F.Cu at (123.8, 146.7)
- added JP9: SolderJumper_2_Open, Jumper:SolderJumper-2_P1.3mm_Open_RoundedPad1.0x1.5mm, F.Cu at (125.8, 105.2)
- JP1, JP8: footprint Jumper:SolderJumper-2_P1.3mm_Bridged_RoundedPad1.0x1.5mm -> Jumper:SolderJumper-2_P1.3mm_Open_RoundedPad1.0x1.5mm
Routing:
- net GND: track 85.9 -> 102.2 mm, vias 107 -> 92
- net ~{SRST}: track 29.1 -> 32.4 mm, vias 1 -> 2
Other:
- board text added: "Boot"
- board text added: "PB0"
- board text added: "PB1"
- board text added: "PB3"
- board text added: "PB4"
- board text added: "PB6"
- board text added: "PB7"
- board text added: "PC0"
- board text added: "PC1"
- board text added: "PC2"
- board text added: "PC3"
- board text added: "PD0"
- board text added: "PD1"
- board text added: "PD2"
- board text added: "PD5"
- board text added: "PD6"
- board text added: "PE1"
- board text added: "RSense"
- board text added: "SRST"
