File: EduboardV2_ATmega328PB.kicad_pcb (KiCad board)
At the start: 4 copper layers, 35 x 63.3 mm, 69 parts, among them J1 EduboardV2 PCIE UP Board Conn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, J2 JTAG_mEDBG, Q3 AO3401A, SW1 K2-1102SP-C4SC-04, U1 ATMEGA32U4-MU, U2 ATMEGA328PB-AUR, U5 LD1117S33TR_SOT223, X1 M16000E067

Commit message: change version to 1.1
Parts:
- removed C25, C27: 4u7, Capacitor_SMD:C_0805_2012Metric
- removed C26, C28: 100n, Capacitor_SMD:C_0402_1005Metric
- removed D1: LESD5D5.0CT1G, EduboardV2_kicadlib:SOD-523_L1.2-W0.8-LS1.6-BI
- removed Q3: AO3401A, EduboardV2_kicadlib:SOT-23_L2.9-W1.3-P1.90-LS2.4-BR
- removed R25: 3k3, Resistor_SMD:R_0402_1005Metric
- removed R31, R32: 0R, Resistor_SMD:R_0603_1608Metric
- removed R6, R7: 10k, Resistor_SMD:R_0402_1005Metric
- removed U5: LD1117S33TR_SOT223, Package_TO_SOT_SMD:SOT-223-3_TabPin2
- removed USBC1: USB3.1C16PFSMT, EduboardV2_kicadlib:USB-C-SMD_TYPE-C-USB-17
- moved SW1 27.0 mm to (104.3, 133.6), turned to 180 degrees
- moved D2 9.99 mm to (103.6, 118.3), turned to 0 degrees
- moved D3 9.98 mm to (106.7, 118.3), turned to 180 degrees
Connections:
- C5 pad 1: Net-(C5-Pad1) -> +3V3
- D2 pad 2: D+ -> USB_Debug_D-
- D3 pad 2: D- -> USB_Debug_D+
- J1 pad 6: 3.3V_Sense -> +3V3
- JP34 pad 1: UART1_RX -> SPI_MISO
- JP34 pad 3: SPI_MISO -> UART1_RX
- R5 pad 2: PROG_SPI_MOSI -> PROG_SPI_MISO
- R8 pad 2: PROG_SPI_MISO -> PROG_SPI_MOSI
- U1 pad 14: Net-(C5-Pad1) -> +3V3
Routing:
- net +3V3: track 150.7 -> 6.15 mm, vias 12 -> 0
- net GND: track 102.2 -> 2.10 mm, vias 92 -> 2
- net VBUS: track 96.8 -> 0.00 mm, vias 4 -> 0
- net RS485_DE: track 53.8 -> 0.00 mm
- net UART1_TX: track 46.2 -> 0.00 mm, vias 1 -> 0
- net UART1_RX: track 44.7 -> 0.00 mm, vias 1 -> 0
- net SPI_MISO: track 43.6 -> 0.00 mm, vias 3 -> 0
- net SPI_SCK: track 40.5 -> 0.00 mm, vias 2 -> 0
- net ~{RESET_DW}: track 40.2 -> 0.00 mm
- net SPI_MOSI: track 39.4 -> 0.00 mm, vias 3 -> 0
- net GPIOX0: track 38.8 -> 0.00 mm
- net GPIO_SW0: track 37.8 -> 0.00 mm, vias 1 -> 0
- net GPIO_WS2812_DATA: track 36.8 -> 0.00 mm, vias 2 -> 0
- net GPIO_RotEnc_B: track 36.6 -> 0.00 mm, vias 2 -> 0
- net GPIO_SW1: track 35.5 -> 0.00 mm, vias 1 -> 0
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
Commit message: arrange parts and layout v1.1.
Parts:
- removed D3: LESD5D5.0CT1G, EduboardV2_kicadlib:SOD-523_L1.2-W0.8-LS1.6-BI
- removed JP16, JP17, JP18, JP19, JP20, JP21, JP22, JP3, JP30, JP34, JP5, JP6, JP7: SolderJumper_3_Bridged12, EduboardV2_kicadlib:SolderJumper_Small-3_bridged12
- removed JP23, JP4: SolderJumper_3_Bridged12, EduboardV2_kicadlib:SolderJumper_Small-4_bridged14
- removed JP8, JP9: SolderJumper_2_Open, Jumper:SolderJumper-2_P1.3mm_Open_RoundedPad1.0x1.5mm
- added D1: LESD5D5.0CT1G, EduboardV2_kicadlib:SOD-523_L1.2-W0.8-LS1.6-BI, F.Cu at (103.6, 118.3)
- added R14: 0R, Resistor_SMD:R_0603_1608Metric, F.Cu at (123.9, 137.5)
- added R15: 0R, Resistor_SMD:R_0603_1608Metric, F.Cu at (114.0, 150.3)
- added R16: 0R, Resistor_SMD:R_0603_1608Metric, F.Cu at (115.5, 150.3)
- added R17: 0R, Resistor_SMD:R_0603_1608Metric, F.Cu at (110.8, 144.2)
- added R18: 0R, Resistor_SMD:R_0603_1608Metric, F.Cu at (110.8, 145.7)
- added R20: 0R, Resistor_SMD:R_0603_1608Metric, F.Cu at (132.3, 148.1)
- added R21: 0R, Resistor_SMD:R_0603_1608Metric, F.Cu at (117.9, 137.5)
- added R22: 0R, Resistor_SMD:R_0603_1608Metric, F.Cu at (114.9, 137.5)
- added R23: 0R, Resistor_SMD:R_0603_1608Metric, F.Cu at (116.4, 137.5)
- added R24: 0R, Resistor_SMD:R_0603_1608Metric, F.Cu at (110.8, 141.2)
- added R25: 0R, Resistor_SMD:R_0603_1608Metric, F.Cu at (110.8, 139.7)
- added R26: 0R, Resistor_SMD:R_0603_1608Metric, F.Cu at (110.8, 142.7)
- added R27: 0R, Resistor_SMD:R_0603_1608Metric, F.Cu at (129.9, 137.5)
- added R28: 1k, Resistor_SMD:R_0402_1005Metric, F.Cu at (123.1, 117.8)
- added R31: 0R, Resistor_SMD:R_0603_1608Metric, F.Cu at (132.3, 146.6)
- added R32: 0R, Resistor_SMD:R_0603_1608Metric, F.Cu at (132.3, 145.1)
- added R33: 0R, Resistor_SMD:R_0603_1608Metric, F.Cu at (110.9, 150.3)
- added R34: 0R, Resistor_SMD:R_0603_1608Metric, F.Cu at (112.4, 150.3)
- added R35: 10k, Resistor_SMD:R_0402_1005Metric, F.Cu at (106.4, 140.2)
- added R36: 3k3, Resistor_SMD:R_0402_1005Metric, F.Cu at (126.0, 109.5)
- added R37: 0R, Resistor_SMD:R_0603_1608Metric, F.Cu at (104.4, 115.0)
- added R38: 0R, Resistor_SMD:R_0603_1608Metric, F.Cu at (105.9, 115.0)
- added R39: 100k, Resistor_SMD:R_0402_1005Metric, F.Cu at (116.0, 115.2)
- added R40: 0R, Resistor_SMD:R_0603_1608Metric, F.Cu at (125.8, 113.7)
- added R41: 330R, Resistor_SMD:R_0603_1608Metric, F.Cu at (109.8, 118.1)
- added R42: 330R, Resistor_SMD:R_0603_1608Metric, F.Cu at (112.8, 118.1)
- added R43: 330R, Resistor_SMD:R_0603_1608Metric, F.Cu at (111.3, 118.1)
- added R44: 330R, Resistor_SMD:R_0603_1608Metric, F.Cu at (123.4, 108.0)
- added R45: 3k3, Resistor_SMD:R_0402_1005Metric, F.Cu at (124.6, 113.7)
- added R46: 100k, Resistor_SMD:R_0402_1005Metric, F.Cu at (125.5, 105.1)
- added R6: 0R, Resistor_SMD:R_0603_1608Metric, F.Cu at (132.3, 143.6)
- added R7: 0R, Resistor_SMD:R_0603_1608Metric, F.Cu at (131.4, 137.5)
- C5: value 100n -> 12p
- C7: value 12p -> 100n
- JP2: value SolderJumper_3_Bridged12 -> SolderJumper_2_Open; footprint EduboardV2_kicadlib:SolderJumper_Small-3_bridged12 -> Jumper:SolderJumper-2_P1.3mm_Open_RoundedPad1.0x1.5mm; moved to F.Cu
- R1, R13: value 100k -> 0R; footprint Resistor_SMD:R_0402_1005Metric -> Resistor_SMD:R_0603_1608Metric
- R10, R9: value 1k -> 0R; footprint Resistor_SMD:R_0402_1005Metric -> Resistor_SMD:R_0603_1608Metric
- R11, R4, R5, R8: value 330R -> 0R
- R12, R2: value 3k3 -> 0R; footprint Resistor_SMD:R_0402_1005Metric -> Resistor_SMD:R_0603_1608Metric
- R19: value 10k -> 0R; footprint Resistor_SMD:R_0402_1005Metric -> Resistor_SMD:R_0603_1608Metric
- R29: value 0R -> 1k; footprint Resistor_SMD:R_0603_1608Metric -> Resistor_SMD:R_0402_1005Metric
- U1: value ATMEGA32U4-MU -> ATMEGA328PB-AUR; footprint EduboardV2_kicadlib:VQFN-44_L7.0-W7.0-P0.50-BL-EP5.2 -> EduboardV2_kicadlib:TQFP-32_L7.0-W7.0-P0.80-LS9.0-BL
- U2: value ATMEGA328PB-AUR -> ATMEGA32U4-MU; footprint EduboardV2_kicadlib:TQFP-32_L7.0-W7.0-P0.80-LS9.0-BL -> EduboardV2_kicadlib:VQFN-44_L7.0-W7.0-P0.50-BL-EP5.2
- moved G*** 45.3 mm to (108.9, 103.9), turned to -90 degrees
- moved JP2 34.6 mm to (126.0, 107.3), turned to -90 degrees
- moved R1 32.6 mm to (111.9, 137.5), turned to -90 degrees
- moved C10 31.8 mm to (120.1, 103.6), turned to 0 degrees
- moved R30 31.8 mm to (128.4, 137.5), turned to -90 degrees
- moved R5 29.3 mm to (132.3, 142.1), turned to 180 degrees
- moved C9 29.2 mm to (114.9, 103.6)
- moved R12 26.4 mm to (122.4, 137.5), turned to 90 degrees
- moved R10 26.3 mm to (133.5, 121.7)
- moved R11 25.5 mm to (120.9, 137.5), turned to -90 degrees
- moved U2 25.5 mm to (117.5, 109.0), turned to -90 degrees
- moved R2 25.5 mm to (113.4, 137.5), turned to -90 degrees
- moved R4 23.4 mm to (126.9, 137.5), turned to -90 degrees
- moved C11 23.3 mm to (122.8, 111.7), turned to 90 degrees
- moved G*** 22.5 mm to (122.2, 145.1), turned to -90 degrees
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Connections:
- C1 pad 1: Net-(U1-UCap) -> +3V3
- C10 pad 1: +3V3 -> GND
- C10 pad 2: GND -> +3V3
- C11 pad 1: +3V3 -> GND
- C11 pad 2: GND -> +3V3
- C2 pad 1: GND -> +3V3
- C2 pad 2: +3V3 -> GND
- C3 pad 1: GND -> +3V3
- C3 pad 2: +3V3 -> GND
- C4 pad 1: GND -> ~{SRST}
- C4 pad 2: +3V3 -> GND
- C5 pad 1: +3V3 -> Net-(U2-XTAL2)
- C6 pad 1: Net-(U1-XTAL2) -> Net-(U2-XTAL1)
- C7 pad 1: Net-(U1-XTAL1) -> Net-(U2-UCap)
- C8 pad 1: ~{SRST} -> +3V3
- C9 pad 1: +3V3 -> GND
- C9 pad 2: GND -> +3V3
- D2 pad 2: USB_Debug_D- -> USB_Debug_D+
- JP1 pad 1: Net-(JP1-A) -> GND
- JP1 pad 2: GND -> ~{SRST}
- JP2 pad 2: UART0_TX -> GND
- R1 pad 1: Net-(JP1-A) -> Net-(U1-(XTAL2/TOSC2)PB7)
- R1 pad 2: +3V3 -> GPIO_RotEnc_SW
- R10 pad 1: Net-(JP3-A) -> EXT_CLK
- R10 pad 2: PROG_UART_TX -> Net-(U1-(XTAL1/TOSC1)PB6)
- R11 pad 1: EXT_CLK -> Net-(U1-(OC1A/PTCXY)PB1)
- R11 pad 2: CLK_OUT -> GPIOX4
- R12 pad 1: STATUS_LED -> GPIO_RotEnc_B
- R12 pad 2: Net-(LED1-C) -> Net-(U1-(SCL1/T4/PTCXY)PE1)
- R13 pad 1: ~{SRST} -> Net-(U1-(OC1A/PTCXY)PB1)
- R13 pad 2: +3V3 -> LCD_DC
- R19 pad 1: +3V3 -> GPIO_LED7
- R19 pad 2: ~{RESET_DW} -> Net-(U1-PD2(PTCXY/INT0/OC3B/OC4B))
- R2 pad 1: ~{RESET_DW} -> Net-(U1-(XTAL2/TOSC2)PB7)
- R2 pad 2: +3V3 -> GPIO_Buzzer
- R29 pad 1: USB_Debug_D- -> UART0_RX
- R29 pad 2: USB_N -> PROG_UART_TX
- R3 pad 1: ~{RESET_DW} -> Net-(U1-(OC0B/T1/PTCXY)PD5)
- R3 pad 2: debugWire -> GPIO_PWM_R
- R30 pad 1: USB_Debug_D+ -> Net-(U1-PC2(ADC2/PTCY))
- R30 pad 2: USB_P -> GPIOX1
- R4 pad 1: SPI_SCK -> Net-(U1-(OC0B/T1/PTCXY)PD5)
- R4 pad 2: PROG_SPI_SCK -> GPIO_LED5
- R5 pad 1: SPI_MISO -> Net-(U1-(OC0A/PTCXY/AIN0)PD6)
- R5 pad 2: PROG_SPI_MISO -> GPIO_PWM_G
- R8 pad 1: SPI_MOSI -> RS485_DE
- R8 pad 2: PROG_SPI_MOSI -> Net-(U1-(XTAL1/TOSC1)PB6)
- R9 pad 1: Net-(JP2-A) -> Net-(U1-(ICP1/CLKO/PTCXY)PB0)
- R9 pad 2: PROG_UART_RX -> GPIO_LED4
- U1 pad 1: debugWire -> GPIO_LED0
- U1 pad 10: PROG_SPI_MOSI -> Net-(U1-(OC0A/PTCXY/AIN0)PD6)
- U1 pad 11: PROG_SPI_MISO -> GPIO_WS2812_DATA
- U1 pad 12: unconnected-(U1-PB7(PCINT7/OC0A/OC1C/RTS#)-Pad12) -> Net-(U1-(ICP1/CLKO/PTCXY)PB0)
- U1 pad 13: ~{SRST} -> Net-(U1-(OC1A/PTCXY)PB1)
- U1 pad 14: +3V3 -> LCD_CS
- U1 pad 15: GND -> UP_SPI_MOSI
- U1 pad 16: Net-(U1-XTAL2) -> UP_SPI_MISO
- U1 pad 17: Net-(U1-XTAL1) -> SPI_SCK
- U1 pad 18: unconnected-(U1-PD0(OC0B/SCL/INT0)-Pad18) -> +3V3
- U1 pad 19: unconnected-(U1-PD1(SDA/INT1)-Pad19) -> GPIO_SW0
- U1 pad 2: VBUS -> GPIO_LED1
- U1 pad 20: PROG_UART_RX -> +3V3
- U1 pad 21: PROG_UART_TX -> GND
- U1 pad 22: unconnected-(U1-PD5(XCK1/CTS#)-Pad22) -> GPIO_SW1
- U1 pad 23: GND -> Net-(U1-PC0(ADC0/PTCY/MISO1))
- U1 pad 24: +3V3 -> Net-(U1-PC1(ADC1/PTCY/SCK1))
- U1 pad 25: debugWire -> Net-(U1-PC2(ADC2/PTCY))
- U1 pad 26: unconnected-(U1-PD6(T1/~{OC4D}/ADC9)-Pad26) -> Net-(U1-PC3(ADC3/PTCY))
- U1 pad 27: unconnected-(U1-PD7(T0/OC4D/ADC10)-Pad27) -> SDA
- U1 pad 28: RESET_SENSE -> SCL
- U1 pad 29: EXT_CLK -> ~{RESET_DW}
- U1 pad 3: USB_N -> GPIO_LED2
- U1 pad 30: POWER_ENABLE -> UART0_RX
- U1 pad 31: STATUS_LED -> UART0_TX
- U1 pad 32: CLK_OUT -> Net-(U1-PD2(PTCXY/INT0/OC3B/OC4B))
- U1 pad 4: USB_P -> +3V3
- U1 pad 6: Net-(U1-UCap) -> Net-(U1-(SCL1/T4/PTCXY)PE1)
- U1 pad 7: VBUS -> Net-(U1-(XTAL1/TOSC1)PB6)
- U1 pad 8: unconnected-(U1-PB0(SS/PCINT0)-Pad8) -> Net-(U1-(XTAL2/TOSC2)PB7)
- U1 pad 9: PROG_SPI_SCK -> Net-(U1-(OC0B/T1/PTCXY)PD5)
- U2 pad 1: GPIO_LED0 -> debugWire
- U2 pad 10: Net-(JP18-C) -> PROG_SPI_MOSI
- U2 pad 11: GPIO_WS2812_DATA -> PROG_SPI_MISO
- U2 pad 12: Net-(JP17-C) -> unconnected-(U2-PB7(PCINT7/OC0A/OC1C/RTS#)-Pad12)
- U2 pad 13: Net-(JP16-C) -> ~{SRST}
- U2 pad 14: LCD_CS -> +3V3
- U2 pad 15: Net-(JP30-C) -> GND
- U2 pad 16: Net-(JP34-C) -> Net-(U2-XTAL2)
- U2 pad 17: SPI_SCK -> Net-(U2-XTAL1)
- U2 pad 18: +3V3 -> unconnected-(U2-PD0(OC0B/SCL/INT0)-Pad18)
- U2 pad 19: GPIO_SW0 -> unconnected-(U2-PD1(SDA/INT1)-Pad19)
- U2 pad 2: GPIO_LED1 -> VBUS
- U2 pad 20: +3V3 -> PROG_UART_RX
- U2 pad 21: GND -> PROG_UART_TX
- U2 pad 22: GPIO_SW1 -> unconnected-(U2-PD5(XCK1/CTS#)-Pad22)
- U2 pad 23: Net-(JP23-C) -> GND
- U2 pad 24: Net-(JP4-C) -> +3V3
- U2 pad 25: Net-(JP5-C) -> debugWire
- U2 pad 26: Net-(JP6-C) -> unconnected-(U2-PD6(T1/~{OC4D}/ADC9)-Pad26)
- U2 pad 27: SDA -> unconnected-(U2-PD7(T0/OC4D/ADC10)-Pad27)
- U2 pad 28: SCL -> RESET_SENSE
- U2 pad 29: ~{RESET_DW} -> EXT_CLK
- U2 pad 3: GPIO_LED2 -> USB_N
- U2 pad 30: UART0_RX -> POWER_ENABLE
- U2 pad 31: UART0_TX -> STATUS_LED
- U2 pad 32: Net-(JP7-C) -> CLK_OUT
- U2 pad 4: +3V3 -> USB_P
- U2 pad 6: Net-(JP21-C) -> Net-(U2-UCap)
- U2 pad 7: Net-(JP22-C) -> VBUS
- U2 pad 8: Net-(JP20-C) -> unconnected-(U2-PB0(SS/PCINT0)-Pad8)
- U2 pad 9: Net-(JP19-C) -> PROG_SPI_SCK
- X1 pad 1: Net-(U1-XTAL1) -> Net-(U2-XTAL1)
- X1 pad 3: Net-(U1-XTAL2) -> Net-(U2-XTAL2)
Routing:
- net +3V3: track 6.15 -> 193.2 mm, vias 0 -> 7
- net GND: track 2.10 -> 86.8 mm, vias 2 -> 64
- net VBUS: track 0.00 -> 67.6 mm, vias 0 -> 2
- net ~{RESET_DW}: track 0.00 -> 54.2 mm, vias 0 -> 3
- net RS485_DE: track 0.00 -> 50.8 mm, vias 0 -> 2
- net SPI_SCK: track 0.00 -> 44.1 mm, vias 0 -> 1
- net GPIO_SW0: track 0.00 -> 43.2 mm, vias 0 -> 2
- net UP_SPI_MOSI: track 0.00 -> 42.7 mm, vias 0 -> 2
- net UART0_TX: track 0.00 -> 42.7 mm, vias 0 -> 4
- net GPIO_SW1: track 0.00 -> 40.9 mm, vias 0 -> 2
- net UART0_RX: track 0.00 -> 40.5 mm, vias 0 -> 5
- net ~{SRST}: track 0.00 -> 38.7 mm, vias 0 -> 1
- net GPIO_WS2812_DATA: track 0.00 -> 35.9 mm, vias 0 -> 2
- net LCD_CS: track 0.00 -> 35.6 mm, vias 0 -> 1
- net UP_SPI_MISO: track 0.00 -> 35.2 mm, vias 0 -> 2
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- added copper zone on In1.Cu, net GND
Other:
- board text added: "AN0"
- board text added: "BUZZ"
- board text added: "ENCSW"
- board text added: "ENC_A"
- board text added: "ENC_B"
- board text added: "FL_CS"
- board text added: "GPIO0"
- board text added: "GPIO1"
- board text added: "GPIO2"
- board text added: "GPIO3"
- board text added: "GPIO4"
- board text added: "LCDDC"
- board text added: "LED3"
- board text added: "LED4"
- board text added: "LED5"
- board text added: "LED6"
- board text added: "LED7"
- board text added: "MISO"
- board text added: "MOSI"
- board text added: "PWMB"
- board text added: "PWMG"
- board text added: "PWMR"
- board text added: "RESET"
- board text added: "SDCS"
- board text added: "SW2"
- board text added: "SW3"
- board text added: "U0RX"
- board text added: "U0TX"
- board text added: "U1RX"
- board text added: "U1TX"
- board text removed: "PB0"
- board text removed: "PB1"
- board text removed: "PB3"
- board text removed: "PB4"
- board text removed: "PB6"
- board text removed: "PB7"
- board text removed: "PC0"
- board text removed: "PC1"
- board text removed: "PC2"
- board text removed: "PC3"
- board text removed: "PD0"
- board text removed: "PD1"
- board text removed: "PD2"
- board text removed: "PD5"
- board text removed: "PD6"
- board text removed: "PE1"
- board text removed: "RSense"
