File: DebugChip.kicad_sch (KiCad schematic)
At the start: 33 parts, among them Q3 AO3401A, U1 ATMEGA32U4-MU, X1 M16000E067

Commit message: schematic done. layout done aswell. Have to check everything trice
Parts:
- added C8: 100n, Capacitor_SMD:C_0402_1005Metric, symbol Device:C
- added J2: JTAG_mEDBG, Connector_PinHeader_2.54mm:PinHeader_2x05_P2.54mm_Vertical, symbol Connector_Generic:Conn_02x05_Odd_Even
- added JP8: SolderJumper_2_Open, Jumper:SolderJumper-2_P1.3mm_Bridged_RoundedPad1.0x1.5mm, symbol Jumper:SolderJumper_2_Open
- added LED1: 19-217/BHC-ZL1M2RY/3T, EduboardV2_kicadlib:LED0603-FD_BLUE, symbol EduboardV2_kicadlib:19-217_BHC-ZL1M2RY_3T
- added R11: 330R, Resistor_SMD:R_0603_1608Metric, symbol Device:R
- added R12: 3k3, Resistor_SMD:R_0402_1005Metric, symbol Device:R
- added R13: 100k, Resistor_SMD:R_0402_1005Metric, symbol Device:R
- C1, C2, C26, C28, C3, C4, C5, C6, C7: footprint Capacitor_SMD:C_0603_1608Metric -> Capacitor_SMD:C_0402_1005Metric
- JP1: footprint (none) -> Jumper:SolderJumper-2_P1.3mm_Bridged_RoundedPad1.0x1.5mm
- R1, R2, R25, R6, R7: footprint Resistor_SMD:R_0603_1608Metric -> Resistor_SMD:R_0402_1005Metric
Connections:
- net +3V3: now also R2.2, J2.4 (Pin_4), LED1.2 (A), R13.2
- net CLK_OUT: now also R11.2
- net EXT_CLK: now also R11.1
- net GND: now also C8.2, J2.10 (Pin_10), J2.2 (Pin_2)
- net RESET_SENSE: now also JP8.2 (B)
- net STATUS_LED: now also R12.1
- net TCK: now also J2.1 (Pin_1)
- net TDI: now also J2.9 (Pin_9)
- net TDO: now also J2.3 (Pin_3)
- net TMS: now also J2.5 (Pin_5)
- net ~{RESET_DW}: now also JP8.1 (A)
- net ~{SRST}: now also C8.1, J2.6 (Pin_6), R13.1
- new net: LED1.1 (C), R12.2
- no-connect marks 11 -> 13

Commit message: ready for order first prototype
Parts:
- added JP9: SolderJumper_2_Open, Jumper:SolderJumper-2_P1.3mm_Open_RoundedPad1.0x1.5mm, symbol Jumper:SolderJumper_2_Open
- J2: now left out of the parts list
- JP1, JP8: footprint Jumper:SolderJumper-2_P1.3mm_Bridged_RoundedPad1.0x1.5mm -> Jumper:SolderJumper-2_P1.3mm_Open_RoundedPad1.0x1.5mm
Connections:
- net GND: now also JP9.1 (A)
- net ~{SRST}: now also JP9.2 (B)
Changed lines of the file:
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@@
+    (stroke (width 0) (type default))
+  )
+  (wire (pts (xy 117.475 36.195) (xy 122.555 36.195))
     (stroke (width 0) (type default))
   )
@@
   )
   (wire (pts (xy 73.025 132.08) (xy 71.755 132.08))
+    (stroke (width 0) (type default))
+  )
+  (wire (pts (xy 117.475 43.815) (xy 117.475 48.26))
     (stroke (width 0) (type default))
   )
@@
       (effects (font (size 1.27 1.27)) hide)
     )
-    (property "Footprint" "Jumper:SolderJumper-2_P1.3mm_Bridged_RoundedPad1.0x1.5mm" (at 269.24 54.61 0)
+    (property "Footprint" "Jumper:SolderJumper-2_P1.3mm_Open_RoundedPad1.0x1.5mm" (at 269.24 54.61 0)
       (effects (font (size 1.27 1.27)) hide)
     )
@@
   )
   (symbol (lib_id "Connector_Generic:Conn_02x05_Odd_Even") (at 87.63 36.195 0) (unit 1)
-    (in_bom yes) (on_board yes) (dnp no) (fields_autoplaced)
+    (in_bom no) (on_board yes) (dnp no) (fields_autoplaced)
     (property "Reference" "J2" (at 88.9 26.035 0)
       (effects (font (size 1.27 1.27)))
@@
     )
   )
+  (symbol (lib_id "Jumper:SolderJumper_2_Open") (at 117.475 40.005 90) (unit 1)
+    (in_bom yes) (on_board yes) (dnp no)
+    (property "Reference" "JP9" (at 114.935 40.005 0)
+      (effects (font (size 1.27 1.27)))
+    )
+    (property "Value" "SolderJumper_2_Open" (at 114.935 40.005 0)
+      (effects (font (size 1.27 1.27)) hide)
+    )
+    (property "Footprint" "Jumper:SolderJumper-2_P1.3mm_Open_RoundedPad1.0x1.5mm" (at 117.475 40.005 0)
+      (effects (font (size 1.27 1.27)) hide)
+    )
+    (property "Datasheet" "~" (at 117.475 40.005 0)
+      (effects (font (size 1.27 1.27)) hide)
+    )
+    (pin "1")
+    (pin "2")
+    (instances
+      (project "EduboardV2_ATmega328PB"
+        (path "/0ef5f433-62f3-413e-ac2a-aa07749066ac/83d3690c-6ff2-4209-82b8-d055572b14ab"
+          (reference "JP9") (unit 1)
+        )
+      )
+    )
+  )
   (symbol (lib_id "Device:C") (at 122.555 41.91 0) (mirror y) (unit 1)
     (in_bom yes) (on_board yes) (dnp no)
@@
         (path "/0ef5f433-62f3-413e-ac2a-aa07749066ac/83d3690c-6ff2-4209-82b8-d055572b14ab"
           (reference "C8") (unit 1)
+        )
+      )
+    )
+  )
+  (symbol (lib_id "power:GND") (at 117.475 48.26 0) (unit 1)
+    (in_bom yes) (on_board yes) (dnp no) (fields_autoplaced)
+    (property "Reference" "#PWR040" (at 117.475 54.61 0)
+      (effects (font (size 1.27 1.27)) hide)
+    )
+    (property "Value" "GND" (at 117.475 53.34 0)
+      (effects (font (size 1.27 1.27)))
+    )
+    (property "Footprint" "" (at 117.475 48.26 0)
+      (effects (font (size 1.27 1.27)) hide)
+    )
+    (property "Datasheet" "" (at 117.475 48.26 0)
+      (effects (font (size 1.27 1.27)) hide)
+    )
+    (pin "1")
+    (instances
+      (project "EduboardV2_ATmega328PB"
+        (path "/0ef5f433-62f3-413e-ac2a-aa07749066ac/83d3690c-6ff2-4209-82b8-d055572b14ab"
+          (reference "#PWR040") (unit 1)
         )
       )
@@
       (effects (font (size 1.27 1.27)) hide)
     )
-    (property "Footprint" "Jumper:SolderJumper-2_P1.3mm_Bridged_RoundedPad1.0x1.5mm" (at 224.79 132.08 0)
-      (effects (font (size 1.27 1.27)) hide)
-    )
+    (property "Footprint" "Jumper:SolderJumper-2_P1.3mm_Open_RoundedPad1.0x1.5mm" (at 224.79 132.08 0)
+      (effects (font (size 1.27 1.27)) hide)
+    )

Commit message: got first prototypes. Found some errors. not yet corrected, but marked.
Other:
- note added: "VCC not connected"
Changed lines of the file:
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@@
     (effects (font (size 1.27 1.27)) (justify left bottom))
+  )
+  (text "VCC not connected\n" (at 139.065 60.96 0)
+    (effects (font (size 1.27 1.27) (color 255 0 0 1)) (justify left bottom))
   )
   (label "D_P" (at 78.74 151.765 0) (fields_autoplaced)

Commit message: remove voltage regulator and change sense input to 3.3V
Parts:
- removed C25, C27: 4u7, Capacitor_SMD:C_0805_2012Metric, symbol Device:C
- removed C26, C28: 100n, Capacitor_SMD:C_0402_1005Metric, symbol Device:C
- removed Q3: AO3401A, EduboardV2_kicadlib:SOT-23_L2.9-W1.3-P1.90-LS2.4-BR, symbol EduboardV2_kicadlib:AO3401A
- removed R25: 3k3, Resistor_SMD:R_0402_1005Metric, symbol Device:R
- removed U?: LD1117S33TR_SOT223, Package_TO_SOT_SMD:SOT-223-3_TabPin2, symbol Regulator_Linear:LD1117S33TR_SOT223

Commit message: remove USBC Connector, but keep the esd protection
Parts:
- removed D1: LESD5D5.0CT1G, EduboardV2_kicadlib:SOD-523_L1.2-W0.8-LS1.6-BI, symbol EduboardV2_kicadlib:LESD5D5.0CT1G
- removed R31, R32: 0R, Resistor_SMD:R_0603_1608Metric, symbol Device:R
- removed R6, R7: 10k, Resistor_SMD:R_0402_1005Metric, symbol Device:R
- removed USBC1: USB3.1C16PFSMT, EduboardV2_kicadlib:USB-C-SMD_TYPE-C-USB-17, symbol EduboardV2_kicadlib:USB3.1C16PFSMT
Connections:
- net D+ is gone; now on net USB_Debug_D-: D2.2
- net D- is gone; now on net USB_Debug_D+: D3.2
- no-connect marks 13 -> 11
Other:
- note removed: "Optional"
- moved on the sheet: R29, R30

Commit message: add VCC to Pin14 of the atmega32u4
Connections:
- net +3V3: now also C5.1, U1.14 (VCC)
Other:
- note removed: "VCC not connected"
Changed lines of the file:
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@@
   (junction (at 236.855 31.75) (diameter 0) (color 0 0 0 0)
+  )
+  (junction (at 172.085 59.69) (diameter 0) (color 0 0 0 0)
   )
   (junction (at 236.855 77.47) (diameter 0) (color 0 0 0 0)
@@
     (stroke (width 0) (type default))
   )
+  (wire (pts (xy 172.085 20.32) (xy 172.085 59.69))
+    (stroke (width 0) (type default))
+  )
   (wire (pts (xy 228.6 116.84) (xy 234.95 116.84))
     (stroke (width 0) (type default))
@@
     (stroke (width 0) (type default))
   )
-  (wire (pts (xy 168.275 59.69) (xy 175.895 59.69))
+  (wire (pts (xy 168.275 59.69) (xy 172.085 59.69))
     (stroke (width 0) (type default))
   )
@@
   )
   (wire (pts (xy 97.79 44.45) (xy 97.79 41.275))
+    (stroke (width 0) (type default))
+  )
+  (wire (pts (xy 172.085 59.69) (xy 175.895 59.69))
     (stroke (width 0) (type default))
   )
@@
     (at 14.605 15.875 0)
     (effects (font (size 1.27 1.27)) (justify left bottom))
-  )
-  (text "VCC not connected\n" (at 139.065 60.96 0)
-    (effects (font (size 1.27 1.27) (color 255 0 0 1)) (justify left bottom))
   )
   (label "D_P" (at 83.82 60.96 0) (fields_autoplaced)
@@
         )
       )
+    )
+  )
+  (symbol (lib_id "power:+3V3") (at 172.085 20.32 0) (unit 1)
+    (in_bom yes) (on_board yes) (dnp no)
+    (property "Reference" "#PWR08" (at 172.085 24.13 0)
+      (effects (font (size 1.27 1.27)) hide)
+    )
+    (property "Value" "+3V3" (at 172.72 16.51 0)
+      (effects (font (size 1.27 1.27)))
+    )
+    (property "Footprint" "" (at 172.085 20.32 0)
+      (effects (font (size 1.27 1.27)) hide)
+    )
+    (property "Datasheet" "" (at 172.085 20.32 0)
+      (effects (font (size 1.27 1.27)) hide)
+    )
+    (pin "1")
+    (instances
+      (project "EduboardV2_ATmega328PB"
+        (path "/0ef5f433-62f3-413e-ac2a-aa07749066ac/83d3690c-6ff2-4209-82b8-d055572b14ab"
+          (reference "#PWR08") (unit 1)
+        )
+      )

Commit message: switch miso/mosi from atmega32u4 to atmega328
Connections:
- net PROG_SPI_MISO: now also R5.2; no longer R8.2
- net PROG_SPI_MOSI: now also R8.2; no longer R5.2
Changed lines of the file:
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@@
     )
   )
-  (global_label "PROG_SPI_MISO" (shape input) (at 168.275 52.07 180) (fields_autoplaced)
+  (global_label "PROG_SPI_MISO" (shape bidirectional) (at 168.275 52.07 180) (fields_autoplaced)
     (effects (font (size 1.27 1.27)) (justify right))
-    (property "Intersheetrefs" "${INTERSHEET_REFS}" (at 150.613 52.07 0)
+    (property "Intersheetrefs" "${INTERSHEET_REFS}" (at 149.5017 52.07 0)
       (effects (font (size 1.27 1.27)) (justify right) hide)
     )
@@
     )
   )
-  (global_label "PROG_SPI_MOSI" (shape input) (at 215.9 119.38 180) (fields_autoplaced)
-    (effects (font (size 1.27 1.27)) (justify right))
-    (property "Intersheetrefs" "${INTERSHEET_REFS}" (at 198.238 119.38 0)
-      (effects (font (size 1.27 1.27)) (justify right) hide)
-    )
-  )
   (global_label "USB_N" (shape bidirectional) (at 168.275 31.75 180) (fields_autoplaced)
     (effects (font (size 1.27 1.27)) (justify right))
@@
     (property "Intersheetrefs" "${INTERSHEET_REFS}" (at 246.5039 121.92 0)
       (effects (font (size 1.27 1.27)) (justify left) hide)
+    )
+  )
+  (global_label "PROG_SPI_MOSI" (shape bidirectional) (at 215.9 121.92 180) (fields_autoplaced)
+    (effects (font (size 1.27 1.27)) (justify right))
+    (property "Intersheetrefs" "${INTERSHEET_REFS}" (at 197.1267 121.92 0)
+      (effects (font (size 1.27 1.27)) (justify right) hide)
     )
   )
@@
     )
   )
-  (global_label "PROG_SPI_MOSI" (shape output) (at 168.275 49.53 180) (fields_autoplaced)
+  (global_label "PROG_SPI_MISO" (shape bidirectional) (at 215.9 119.38 180) (fields_autoplaced)
     (effects (font (size 1.27 1.27)) (justify right))
-    (property "Intersheetrefs" "${INTERSHEET_REFS}" (at 150.613 49.53 0)
+    (property "Intersheetrefs" "${INTERSHEET_REFS}" (at 197.1267 119.38 0)
+      (effects (font (size 1.27 1.27)) (justify right) hide)
+    )
+  )
+  (global_label "PROG_SPI_MOSI" (shape bidirectional) (at 168.275 49.53 180) (fields_autoplaced)
+    (effects (font (size 1.27 1.27)) (justify right))
+    (property "Intersheetrefs" "${INTERSHEET_REFS}" (at 149.5017 49.53 0)
       (effects (font (size 1.27 1.27)) (justify right) hide)
     )
@@
       (effects (font (size 1.27 1.27)) (justify right) hide)
     )
-  )
-  (global_label "PROG_SPI_MISO" (shape output) (at 215.9 121.92 180) (fields_autoplaced)
-    (effects (font (size 1.27 1.27)) (justify right))
-    (property "Intersheetrefs" "${INTERSHEET_REFS}" (at 198.238 121.92 0)
-      (effects (font (size 1.27 1.27)) (justify right) hide)
-    )
