File: DebugChip.kicad_sch (KiCad schematic)
At the start: 28 parts, among them J2 JTAG_mEDBG, U1 ATMEGA32U4-MU, X1 M16000E067

Commit message: arrange parts and layout v1.1.
Parts:
- removed JP8: SolderJumper_2_Open, Jumper:SolderJumper-2_P1.3mm_Open_RoundedPad1.0x1.5mm, symbol Jumper:SolderJumper_2_Open
- renumbered C2 to C10, C3 to C11, C8 to C4, C6 to C5, C7 to C6, C1 to C7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
Connections:
- net SPI_MISO renamed UP_SPI_MISO
- net SPI_MOSI renamed UP_SPI_MOSI
